File: Hardware/PiGarage.kicad_pcb (KiCad board)
At the start: 2 copper layers, 65 x 56 mm, 78 parts, among them J1 Conn_02x03_Odd_Even, J2 Conn_02x02_Counter_Clockwise, J3 PJ-320B, J4 Conn_02x20_Odd_Even, Q1 AO4407A, Q2 MMBT3904, U1 TPS54560BQDDARQ1, U2 TL431DBZ, U3 PCM5122PWR, U4 AP2112K-3.3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

Commit message: Add J5 JST SH 1.0mm fan output connector
Adds a 2-pin JST SH 1.0mm (BM02B-SRSS-TB) fan power header to the schematic.
Pin 1 = +5V, Pin 2 = GND. Taps the unfiltered 5V rail near U1 (buck converter)
for a 25mm cooling fan. Same connector family as the RPi 5 fan.

Updated docs: README features list, BOM/design-notes.txt (new J5 section,
hand-solder list), and Docs/ordering-guide.md (hand-solder step).
Parts:
- added J5: Conn_01x02_Pin, Connector_JST:JST_SH_BM02B-SRSS-TB_1x02-1MP_P1.00mm_Vertical, F.Cu at (86.5, 44.0)
Routing:
- net +5V: track 78.9 -> 81.7 mm

Commit message: Swap J5 fan connector: JST SH 1.0mm SMD → JST PH 2.0mm through-hole
B2B-PH-K-S (C131337) replaces BM02B-SRSS-TB. Through-hole, keyed,
locking tab — better suited to automotive vibration. Relocated J5
near U1/L1 so fan sits directly over the buck converter hotspot.
Mating: PHR-2 housing + SPH-002T-P0.5L contacts.

Updated schematic footprint, PCB layout, BOM design-notes, and
ordering guide. Notes that C131337 is Extended (~$3 fee) so
hand-soldering is recommended over JLCPCB assembly for this part.
Parts:
- J5: footprint Connector_JST:JST_SH_BM02B-SRSS-TB_1x02-1MP_P1.00mm_Vertical -> Connector_JST:JST_PH_B2B-PH-K_1x02_P2.00mm_Vertical
- moved J5 32.6 mm to (119.0, 41.0), turned to 0 degrees
- moved R4 4.72 mm to (127.5, 40.5), turned to 90 degrees
- moved R3 2.69 mm to (126.0, 40.5), turned to 90 degrees
Connections:
- R5 pad 2: Net-(D1-A1) -> +VBAT
Routing:
- net Net-(U1-FB): track 20.4 -> 17.3 mm
- net +5V: track 81.7 -> 82.8 mm
